File: KiCad_Files/Peripherals.sch (KiCad schematic (older format))
At the start: 24 parts, among them J8 MEM2075-00-140-01-A, J9 Conn_01x02_Male, Q1 PMT280ENEAX, U6 W25Q32JVSSIQ_TR, U7 TCAN330G

Commit message: Add shapes3D folder
Now all 3D models for the components are stored in a single folder, thanks to the Archive Plugin from https://github.com/MitjaNemec/Kicad_action_plugins.git
Parts:
- C19, C20, C26, C27, C28, C29, C30, C31, C32: symbol Device:C_Small -> archive:Device_C_Small
- D4: symbol dk_TVS-Diodes:PESD2CAN_215 -> archive:dk_TVS-Diodes_PESD2CAN_215
- J8: symbol SamacSys_Parts:MEM2075-00-140-01-A -> archive:SamacSys_Parts_MEM2075-00-140-01-A
- J9: symbol Connector:Conn_01x02_Male -> archive:Connector_Conn_01x02_Male
- Q1: symbol SamacSys_Parts:PMT280ENEAX -> archive:SamacSys_Parts_PMT280ENEAX
- R10, R16, R17, R18, R19, R20, R9: symbol Device:R_Small -> archive:Device_R_Small
- RN1, RN2: symbol Device:R_Pack04 -> archive:Device_R_Pack04
- U6: symbol dk_Memory:W25Q32JVSSIQ_TR -> archive:dk_Memory_W25Q32JVSSIQ_TR
- U7: symbol Interface_CAN_LIN:TCAN330G -> archive:Interface_CAN_LIN_TCAN330G
Changed lines of the file:
@@
 $EndDescr
 $Comp
-L power:+3.3V #PWR0139
+L archive:power_+3.3V #PWR0139
 U 1 1 616DD3D7
 P 4200 5175
@@
 	4200 5175 4200 5250
 $Comp
-L power:GND #PWR0140
+L archive:power_GND #PWR0140
 U 1 1 616E5BF7
 P 4200 6900
@@
 	4200 6900 4200 6850
 $Comp
-L Device:R_Pack04 RN2
+L archive:Device_R_Pack04 RN2
 U 1 1 616ED35C
 P 3150 5575
@@
 	3350 5375 3350 5325
 $Comp
-L power:+3.3V #PWR0141
+L archive:power_+3.3V #PWR0141
 U 1 1 616ED34A
 P 3200 5250
@@
 $EndComp
 $Comp
-L Device:R_Pack04 RN1
+L archive:Device_R_Pack04 RN1
 U 1 1 616D8B8F
 P 2675 5575
@@
 	2875 5375 2875 5325
 $Comp
-L power:+3.3V #PWR0142
+L archive:power_+3.3V #PWR0142
 U 1 1 616DBD2E
 P 2725 5250
@@
 $EndComp
 $Comp
-L Device:C_Small C19
+L archive:Device_C_Small C19
 U 1 1 616FE025
 P 4400 5400
@@
 Connection ~ 4200 5250
 $Comp
-L power:GND #PWR0144
+L archive:power_GND #PWR0144
 U 1 1 616FF326
 P 4400 5600
@@
 SD_CARD_CD
 $Comp
-L Connector:Conn_01x02_Male J9
+L archive:Connector_Conn_01x02_Male J9
 U 1 1 6140C721
 P 9525 1750
@@
 $EndComp
 $Comp
-L power:+BATT #PWR0145
+L archive:power_+BATT #PWR0145
 U 1 1 614100DB
 P 9225 1500
@@
 $EndComp
 $Comp
-L SamacSys_Parts:PMT280ENEAX Q1
+L archive:SamacSys_Parts_PMT280ENEAX Q1
 U 1 1 61410D8C
 P 9175 2250
@@
 	9225 1850 9325 1850
 $Comp
-L power:GND #PWR0146
+L archive:power_GND #PWR0146
 U 1 1 614207CC
 P 9225 2800
@@
 $EndComp
 $Comp
-L Device:R_Small R9
+L archive:Device_R_Small R9
 U 1 1 61422276
 P 8575 2350
@@
 $EndComp
 $Comp
-L Device:R_Small R10
+L archive:Device_R_Small R10
 U 1 1 61423B8A
 P 8775 2550
@@
 	9225 2700 9225 2800
 $Comp
-L dk_Memory:W25Q32JVSSIQ_TR U6
+L archive:dk_Memory_W25Q32JVSSIQ_TR U6
 U 1 1 614419FF
 P 9225 5400
@@
 $EndComp
 $Comp
-L power:+3.3V #PWR0147
+L archive:power_+3.3V #PWR0147
 U 1 1 6144F897
 P 9175 4500
@@
 $EndComp
 $Comp
-L Device:C_Small C26
+L archive:Device_C_Small C26
 U 1 1 6144FF8B
 P 9325 4700
@@
 $EndComp
 $Comp
-L power:GND #PWR0148
+L archive:power_GND #PWR0148
 U 1 1 61450343
 P 9325 4850
@@
 Connection ~ 9175 4550
 $Comp
-L power:GND #PWR0149
+L archive:power_GND #PWR0149
 U 1 1 6145B8A8
 P 9175 5900
@@
 	9175 5900 9175 5800
 $Comp
-L Device:R_Small R16
+L archive:Device_R_Small R16
 U 1 1 6145D636
 P 8675 4875
@@
 	9525 5450 9600 5450
 $Comp
-L Device:C_Small C20
+L archive:Device_C_Small C20
 U 1 1 61EAA5F8
 P 4775 5400
@@
 	4200 5250 4200 5650
 $Comp
-L SamacSys_Parts:MEM2075-00-140-01-A J8
+L archive:SamacSys_Parts_MEM2075-00-140-01-A J8
 U 1 1 616CDB72
 P 3550 5950
@@
 	3150 5325 3050 5325
 $Comp
-L power:+3.3V #PWR0160
+L archive:power_+3.3V #PWR0160
 U 1 1 61595989
 P 9600 5225
@@
 	9600 5225 9600 5350
 $Comp
-L Interface_CAN_LIN:TCAN330G U7
+L archive:Interface_CAN_LIN_TCAN330G U7
 U 1 1 61FFDC40
 P 2975 2525
@@
 $EndComp
 $Comp
-L power:+3.3V #PWR0161
+L archive:power_+3.3V #PWR0161
 U 1 1 620360A4
 P 2975 1525
@@
 $EndComp
 $Comp
-L Device:C_Small C28
+L archive:Device_C_Small C28
 U 1 1 620360AA
 P 3175 1725
@@
 	3175 1575 3175 1625
 $Comp
-L power:GND #PWR0162
+L archive:power_GND #PWR0162
 U 1 1 620360B2
 P 3175 1925
@@
 $EndComp
 $Comp
-L Device:C_Small C29
+L archive:Device_C_Small C29
 U 1 1 620360B8
 P 3550 1725
@@
 	2975 3000 2975 2925
 $Comp
-L power:GND #PWR0163
+L archive:power_GND #PWR0163
 U 1 1 6203C3B0
 P 2975 3000
@@
 $EndComp
 $Comp
-L Device:R_Small R17
+L archive:Device_R_Small R17
 U 1 1 620499E0
 P 2175 1975
@@
 $EndComp
 $Comp
-L Device:R_Small R18
+L archive:Device_R_Small R18
 U 1 1 620499E6
 P 2175 2075
@@
 CAN_RXD
 $Comp
-L Device:C_Small C27
+L archive:Device_C_Small C27
 U 1 1 620499EE
 P 1950 2250
@@
 $EndComp
 $Comp
-L power:GND #PWR0164
+L archive:power_GND #PWR0164
 U 1 1 620499F4
 P 1950 2375
@@
 CAN_H
 $Comp
-L Device:R_Small R19
+L archive:Device_R_Small R19
 U 1 1 62072AC4
 P 3700 2350
@@
 $EndComp
 $Comp
-L Device:R_Small R20
+L archive:Device_R_Small R20
 U 1 1 62072ACA
 P 3700 2750
@@
 	3700 2550 3700 2650
 $Comp
-L Device:C_Small C32
+L archive:Device_C_Small C32
 U 1 1 62072AD8
 P 4325 3100
@@
 $EndComp
 $Comp
-L power:GND #PWR0165
+L archive:power_GND #PWR0165
 U 1 1 62072ADE
 P 4325 3225
@@
 	3975 2550 3700 2550
 $Comp
-L power:GND #PWR0166
+L archive:power_GND #PWR0166
 U 1 1 62072AE8
 P 3975 2775
@@
 $EndComp
 $Comp
-L Device:C_Small C30
+L archive:Device_C_Small C30
 U 1 1 62072AEE
 P 3975 2675
@@
 CAN_L
 $Comp
-L power:GND #PWR0167
+L archive:power_GND #PWR0167
 U 1 1 62072B00
 P 4325 2425
@@
 	4325 2425 4325 2400
 $Comp
-L Device:C_Small C31
+L archive:Device_C_Small C31
 U 1 1 62072B07
 P 4325 2300
@@
 	3700 2150 4325 2150
 $Comp
-L dk_TVS-Diodes:PESD2CAN_215 D4
+L archive:dk_TVS-Diodes_PESD2CAN_215 D4
 U 1 1 62072B1A
 P 4975 2550
@@
 	4625 2950 5250 2950
 $Comp
-L power:GND #PWR0168
+L archive:power_GND #PWR0168
 U 1 1 62072B28
 P 5350 2600
